File: hardware/Display Board/open_g_db.kicad_pcb (KiCad board)
At the start: 4 copper layers, 200 x 35 mm, 117 parts, among them IC1 TS04-66-75-BK-160-SMT, IC2 TS04-66-75-BK-160-SMT, J1 DE9_Socket, J2 2-1825027-0, Q1 BC548A, Q10 BC548A, Q11 BC548A, Q12 BC548A, Q13 BC548A, Q14 BC548A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

Commit message: added README and minor changes
Changed lines of the file:
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@@
 	(gr_text "OpenG Project\nDisplay Board\nv1.0 06/2025"
 		(at 230 93 0)
-		(layer "F.Cu")
+		(layer "F.SilkS")
 		(effects
 			(font
