File: hardware/Display Board/Portexpander_LED.kicad_sch (KiCad schematic)
At the start: 69 parts, among them Q10 BC548A, Q11 BC548A, Q12 BC548A, Q13 BC548A, Q14 BC548A, Q2 BC548A, Q3 BC548A, Q4 BC548A, Q5 BC548A, Q6 BC548A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

Commit message: added gerbers and initial for firmware; changed README
Parts:
- D10, D11, D12, D13, D14, D15: Supplier https://www.mouser.de/ProductDetail/Kingbright/WP710A10SGC?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 -> https://www.mouser.de/ProductDetail/Kingbright/WP710A10NC?q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
- D16: Supplier https://www.mouser.de/ProductDetail/Kingbright/WP710A10SGC?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 -> https://www.mouser.de/ProductDetail/Kingbright/WP710A10EC?q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
Changed lines of the file:
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@@
 			)
 		)
-		(property "Datasheet" "https://www.mouser.de/datasheet/2/216/WP710A10SGC-50126.pdf"
+		(property "Datasheet" "https://www.mouser.de/datasheet/2/216/WP710A10NC-232010.pdf"
 			(at 168.91 104.14 0)
 			(effects
@@
 			)
 		)
-		(property "Supplier" "https://www.mouser.de/ProductDetail/Kingbright/WP710A10SGC?qs=sGAEpiMZZMv0DJfhVcWlK512OlMuG%252BmKJmTyC6LM61Bi%252BQ62PTBqPw%3D%3D"
+		(property "Supplier" "https://www.mouser.de/ProductDetail/Kingbright/WP710A10NC?qs=sGAEpiMZZMv0DJfhVcWlK512OlMuG%252BmKmOWyi9B6XRjq9697RCnSRg%3D%3D"
 			(at 168.91 104.14 90)
 			(effects
@@
 			)
 		)
-		(property "Datasheet" "https://www.mouser.de/datasheet/2/216/WP710A10SGC-50126.pdf"
+		(property "Datasheet" "https://www.mouser.de/datasheet/2/216/WP710A10EC-68022.pdf"
 			(at 269.24 104.14 0)
 			(effects
@@
 			)
 		)
-		(property "Supplier" "https://www.mouser.de/ProductDetail/Kingbright/WP710A10SGC?qs=sGAEpiMZZMv0DJfhVcWlK512OlMuG%252BmKJmTyC6LM61Bi%252BQ62PTBqPw%3D%3D"
+		(property "Supplier" "https://www.mouser.de/ProductDetail/Kingbright/WP710A10EC?qs=sGAEpiMZZMv0DJfhVcWlK512OlMuG%252BmKyj5PXr9sewS6qtVgMhus8g%3D%3D"
 			(at 269.24 104.14 90)
 			(effects
@@
 			)
 		)
-		(property "Datasheet" "https://www.mouser.de/datasheet/2/216/WP710A10SGC-50126.pdf"
+		(property "Datasheet" "https://www.mouser.de/datasheet/2/216/WP710A10NC-232010.pdf"
 			(at 219.71 104.14 0)
 			(effects
@@
 			)
 		)
-		(property "Supplier" "https://www.mouser.de/ProductDetail/Kingbright/WP710A10SGC?qs=sGAEpiMZZMv0DJfhVcWlK512OlMuG%252BmKJmTyC6LM61Bi%252BQ62PTBqPw%3D%3D"
+		(property "Supplier" "https://www.mouser.de/ProductDetail/Kingbright/WP710A10NC?qs=sGAEpiMZZMv0DJfhVcWlK512OlMuG%252BmKmOWyi9B6XRjq9697RCnSRg%3D%3D"
 			(at 219.71 104.14 90)
 			(effects
@@
 			)
 		)
-		(property "Datasheet" "https://www.mouser.de/datasheet/2/216/WP710A10SGC-50126.pdf"
+		(property "Datasheet" "https://www.mouser.de/datasheet/2/216/WP710A10NC-232010.pdf"
 			(at 194.31 104.14 0)
 			(effects
@@
 			)
 		)
-		(property "Supplier" "https://www.mouser.de/ProductDetail/Kingbright/WP710A10SGC?qs=sGAEpiMZZMv0DJfhVcWlK512OlMuG%252BmKJmTyC6LM61Bi%252BQ62PTBqPw%3D%3D"
+		(property "Supplier" "https://www.mouser.de/ProductDetail/Kingbright/WP710A10NC?qs=sGAEpiMZZMv0DJfhVcWlK512OlMuG%252BmKmOWyi9B6XRjq9697RCnSRg%3D%3D"
 			(at 194.31 104.14 90)
 			(effects
@@
 			)
 		)
-		(property "Datasheet" "https://www.mouser.de/datasheet/2/216/WP710A10SGC-50126.pdf"
+		(property "Datasheet" "https://www.mouser.de/datasheet/2/216/WP710A10NC-232010.pdf"
 			(at 245.11 104.14 0)
 			(effects
@@
 			)
 		)
-		(property "Supplier" "https://www.mouser.de/ProductDetail/Kingbright/WP710A10SGC?qs=sGAEpiMZZMv0DJfhVcWlK512OlMuG%252BmKJmTyC6LM61Bi%252BQ62PTBqPw%3D%3D"
+		(property "Supplier" "https://www.mouser.de/ProductDetail/Kingbright/WP710A10NC?qs=sGAEpiMZZMv0DJfhVcWlK512OlMuG%252BmKmOWyi9B6XRjq9697RCnSRg%3D%3D"
 			(at 245.11 104.14 90)
 			(effects
@@
 			)
 		)
-		(property "Datasheet" "https://www.mouser.de/datasheet/2/216/WP710A10SGC-50126.pdf"
+		(property "Datasheet" "https://www.mouser.de/datasheet/2/216/WP710A10NC-232010.pdf"
 			(at 116.84 104.14 0)
 			(effects
@@
 			)
 		)
-		(property "Supplier" "https://www.mouser.de/ProductDetail/Kingbright/WP710A10SGC?qs=sGAEpiMZZMv0DJfhVcWlK512OlMuG%252BmKJmTyC6LM61Bi%252BQ62PTBqPw%3D%3D"
+		(property "Supplier" "https://www.mouser.de/ProductDetail/Kingbright/WP710A10NC?qs=sGAEpiMZZMv0DJfhVcWlK512OlMuG%252BmKmOWyi9B6XRjq9697RCnSRg%3D%3D"
 			(at 116.84 104.14 90)
 			(effects
@@
 			)
 		)
-		(property "Datasheet" "https://www.mouser.de/datasheet/2/216/WP710A10SGC-50126.pdf"
+		(property "Datasheet" "https://www.mouser.de/datasheet/2/216/WP710A10NC-232010.pdf"
 			(at 143.51 104.14 0)
 			(effects
@@
 			)
 		)
-		(property "Supplier" "https://www.mouser.de/ProductDetail/Kingbright/WP710A10SGC?qs=sGAEpiMZZMv0DJfhVcWlK512OlMuG%252BmKJmTyC6LM61Bi%252BQ62PTBqPw%3D%3D"
+		(property "Supplier" "https://www.mouser.de/ProductDetail/Kingbright/WP710A10NC?qs=sGAEpiMZZMv0DJfhVcWlK512OlMuG%252BmKmOWyi9B6XRjq9697RCnSRg%3D%3D"
 			(at 143.51 104.14 90)
 			(effects
