File: hardware/Sensor Board/open_g.kicad_pcb (KiCad board)
At the start: 4 copper layers, 65 x 100 mm, 63 parts, among them IC1 TS04-66-75-BK-160-SMT, IC2 TS04-66-75-BK-160-SMT, IC3 5525DSO-DB001DS, J1 DE9_Socket, J2 DM3CS-SF, J3 Conn_01x09_Socket, J4 Conn_01x05_Socket, J5 1861975, U1 ESP32-WROOM-32E

Commit message: added README and minor changes
Changed lines of the file:
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@@
 	(gr_text "OpenG Project\nSensor Board\nv1.0 06/2025"
 		(at 109.4 70.8 90)
-		(layer "F.Cu")
+		(layer "F.SilkS")
 		(effects
 			(font
