File: hardware/Sensor Board/open_g.kicad_sch (KiCad schematic)
At the start: 63 parts, among them IC1 TS04-66-75-BK-160-SMT, IC2 TS04-66-75-BK-160-SMT, IC3 5525DSO-DB001DS, J1 DE9_Socket, J2 DM3CS-SF, J3 Conn_01x09_Socket, J4 Conn_01x05_Socket, J5 1861975, U1 ESP32-WROOM-32E

Commit message: added README and minor changes
Other:
- note removed: "TODO: - UART Pull"
Changed lines of the file:
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@@
-		)
-	)
-	(text "TODO: \n- UART Pull"
-		(exclude_from_sim no)
-		(at 161.29 169.672 0)
-		(effects
-			(font
-				(size 1.27 1.27)
-			)
-			(justify left)
 		)
 	)

Commit message: added gerbers and initial for firmware; changed README
Other:
- note added: "ISM330DHCX Addr: 0x6A"
- note removed: "ISM330DHCX Addr: 0x6A/0x6B"
Changed lines of the file:
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@@
 		)
 	)
-	(text "ISM330DHCX\nAddr: 0x6A/0x6B"
+	(text "ISM330DHCX\nAddr: 0x6A"
 		(exclude_from_sim no)
 		(at 82.55 115.824 0)
